File: flexmag.kicad_sch (KiCad schematic)
At the start: 7 parts, among them J1 Conn_01x06_Male, J2 Conn_01x06_Male, U1 AS5600-ASOM

Commit message: Perfect is the enemy of done
Connections:
- net +5V: now also J1.5 (Pin_5), J2.5 (Pin_5); no longer J1.6 (Pin_6), J2.6 (Pin_6)
- net GND: now also J1.6 (Pin_6), J2.6 (Pin_6); no longer J1.5 (Pin_5), J2.5 (Pin_5)
- net Aout: now reaches U1.3 (OUT)
- net PGO: now reaches U1.5 (PGO)
Changed lines of the file:
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@@
     (stroke (width 0) (type default) (color 0 0 0 0))
   )
-  (wire (pts (xy 88.9 39.37) (xy 88.9 48.26))
+  (wire (pts (xy 90.17 39.37) (xy 90.17 48.26))
     (stroke (width 0) (type default) (color 0 0 0 0))
   )
@@
     (stroke (width 0) (type default) (color 0 0 0 0))
   )
+  (wire (pts (xy 127 52.07) (xy 130.81 52.07))
+    (stroke (width 0) (type default) (color 0 0 0 0))
+  )
   (wire (pts (xy 130.81 59.69) (xy 121.92 59.69))
     (stroke (width 0) (type default) (color 0 0 0 0))
   )
-  (wire (pts (xy 129.54 52.07) (xy 130.81 52.07))
-    (stroke (width 0) (type default) (color 0 0 0 0))
-  )
   (wire (pts (xy 110.49 44.45) (xy 105.41 44.45))
     (stroke (width 0) (type default) (color 0 0 0 0))
@@
     (stroke (width 0) (type default) (color 0 0 0 0))
   )
-  (wire (pts (xy 129.54 63.5) (xy 129.54 52.07))
+  (wire (pts (xy 129.54 49.53) (xy 129.54 63.5))
     (stroke (width 0) (type default) (color 0 0 0 0))
   )
@@
     (stroke (width 0) (type default) (color 0 0 0 0))
   )
-  (wire (pts (xy 132.08 74.93) (xy 132.08 77.47))
-    (stroke (width 0) (type default) (color 0 0 0 0))
-  )
-  (wire (pts (xy 132.08 95.25) (xy 132.08 80.01))
+  (wire (pts (xy 129.54 74.93) (xy 129.54 80.01))
+    (stroke (width 0) (type default) (color 0 0 0 0))
+  )
+  (wire (pts (xy 129.54 80.01) (xy 134.62 80.01))
+    (stroke (width 0) (type default) (color 0 0 0 0))
+  )
+  (wire (pts (xy 132.08 77.47) (xy 132.08 95.25))
     (stroke (width 0) (type default) (color 0 0 0 0))
   )
@@
     (stroke (width 0) (type default) (color 0 0 0 0))
   )
-  (wire (pts (xy 132.08 80.01) (xy 134.62 80.01))
-    (stroke (width 0) (type default) (color 0 0 0 0))
-  )
-  (wire (pts (xy 129.54 46.99) (xy 129.54 49.53))
+  (wire (pts (xy 48.26 44.45) (xy 52.07 44.45))
     (stroke (width 0) (type default) (color 0 0 0 0))
   )
@@
     (stroke (width 0) (type default) (color 0 0 0 0))
   )
-  (wire (pts (xy 82.55 39.37) (xy 88.9 39.37))
+  (wire (pts (xy 82.55 46.99) (xy 85.09 46.99))
+    (stroke (width 0) (type default) (color 0 0 0 0))
+  )
+  (wire (pts (xy 132.08 77.47) (xy 134.62 77.47))
+    (stroke (width 0) (type default) (color 0 0 0 0))
+  )
+  (wire (pts (xy 82.55 39.37) (xy 90.17 39.37))
     (stroke (width 0) (type default) (color 0 0 0 0))
   )
@@
     (stroke (width 0) (type default) (color 0 0 0 0))
   )
-  (wire (pts (xy 132.08 77.47) (xy 134.62 77.47))
+  (wire (pts (xy 127 46.99) (xy 127 52.07))
     (stroke (width 0) (type default) (color 0 0 0 0))
   )
@@
   (wire (pts (xy 25.4 38.1) (xy 25.4 39.37))
     (stroke (width 0) (type default) (color 0 0 0 0))
+  )
+  (label "PGO" (at 85.09 46.99 0)
+    (effects (font (size 1.27 1.27)) (justify left bottom))
+  )
+  (label "Aout" (at 48.26 44.45 0)
+    (effects (font (size 1.27 1.27)) (justify left bottom))
   )
   (symbol (lib_id "AS5600:AS5600-ASOM") (at 52.07 39.37 0) (unit 1)
@@
     (pin "2")
   )
-  (symbol (lib_id "power:+5V") (at 129.54 46.99 0) (unit 1)
-    (in_bom yes) (on_board yes) (fields_autoplaced)
-    (property "Reference" "#PWR05" (id 0) (at 129.54 50.8 0)
-      (effects (font (size 1.27 1.27)) hide)
-    )
-    (property "Value" "+5V" (id 1) (at 129.54 41.91 0))
-    (property "Footprint" "" (id 2) (at 129.54 46.99 0)
-      (effects (font (size 1.27 1.27)) hide)
-    )
-    (property "Datasheet" "" (id 3) (at 129.54 46.99 0)
-      (effects (font (size 1.27 1.27)) hide)
-    )
-    (pin "1")
-  )
-  (symbol (lib_id "power:+5V") (at 132.08 74.93 0) (unit 1)
-    (in_bom yes) (on_board yes) (fields_autoplaced)
-    (property "Reference" "#PWR07" (id 0) (at 132.08 78.74 0)
-      (effects (font (size 1.27 1.27)) hide)
-    )
-    (property "Value" "+5V" (id 1) (at 132.08 69.85 0))
-    (property "Footprint" "" (id 2) (at 132.08 74.93 0)
-      (effects (font (size 1.27 1.27)) hide)
-    )
-    (property "Datasheet" "" (id 3) (at 132.08 74.93 0)
+  (symbol (lib_id "power:+5V") (at 127 46.99 0) (unit 1)
+    (in_bom yes) (on_board yes) (fields_autoplaced)
+    (property "Reference" "#PWR05" (id 0) (at 127 50.8 0)
+      (effects (font (size 1.27 1.27)) hide)
+    )
+    (property "Value" "+5V" (id 1) (at 127 41.91 0))
+    (property "Footprint" "" (id 2) (at 127 46.99 0)
+      (effects (font (size 1.27 1.27)) hide)
+    )
+    (property "Datasheet" "" (id 3) (at 127 46.99 0)
+      (effects (font (size 1.27 1.27)) hide)
+    )
+    (pin "1")
+  )
+  (symbol (lib_id "power:+5V") (at 129.54 74.93 0) (unit 1)
+    (in_bom yes) (on_board yes)
+    (property "Reference" "#PWR07" (id 0) (at 129.54 78.74 0)
+      (effects (font (size 1.27 1.27)) hide)
+    )
+    (property "Value" "+5V" (id 1) (at 129.54 71.12 0))
+    (property "Footprint" "" (id 2) (at 129.54 74.93 0)
+      (effects (font (size 1.27 1.27)) hide)
+    )
+    (property "Datasheet" "" (id 3) (at 129.54 74.93 0)
       (effects (font (size 1.27 1.27)) hide)
     )
@@
     (pin "2")
   )
-  (symbol (lib_id "power:GND") (at 88.9 48.26 0) (unit 1)
-    (in_bom yes) (on_board yes) (fields_autoplaced)
-    (property "Reference" "#PWR03" (id 0) (at 88.9 54.61 0)
-      (effects (font (size 1.27 1.27)) hide)
-    )
-    (property "Value" "GND" (id 1) (at 88.9 53.34 0))
-    (property "Footprint" "" (id 2) (at 88.9 48.26 0)
-      (effects (font (size 1.27 1.27)) hide)
-    )
-    (property "Datasheet" "" (id 3) (at 88.9 48.26 0)
-      (effects (font (size 1.27 1.27)) hide)
-    )
+  (symbol (lib_id "power:GND") (at 90.17 48.26 0) (unit 1)
+    (in_bom yes) (on_board yes) (fields_autoplaced)
+    (property "Reference" "#PWR03" (id 0) (at 90.17 54.61 0)
+      (effects (font (size 1.27 1.27)) hide)
+    )
+    (property "Value" "GND" (id 1) (at 90.17 53.34 0))
+    (property "Footprint" "" (id 2) (at 90.17 48.26 0)
+      (effects (font (size 1.27 1.27)) hide)
+    )
+    (property "Datasheet" "" (id 3) (at 90.17 48.26 0)
+      (effects (font (size 1.27 1.27)) hide)
+    )
